File: 24v-buck-converter-v1.kicad_pcb (KiCad board)
At the start: 2 copper layers, 44 x 22 mm, 20 parts, among them J1 Conn_01x02, J2 Conn_01x02, J3 Conn_01x02, U1 12V, U2 5V

Commit message: Ensure logo and modules are included
Parts:
- G*** (x2): footprint on-prem:on-prem-logo -> hw-micropow:on-prem-logo
